File: hardware/logicboard/mm-001.brd (EAGLE design)
At the start: 91 x 57 mm, 31 parts, among them IC1 74ALS05N, IC2 LTC485N, IC3 LTC485N, J0 DC5V, J7 DIN5, J8 DIN5, J9 DIN5, X7 NELTRON-7810-XPXC, X9 NELTRON-7810-XPXC

Commit message: Trying to fit in to the new platform.
Parts:
- removed J0: DC5V, con-jack:SPC4077
- removed J7, J8, J9: DIN5, SparkFun-Connectors:DIN5-RA-PTH
- removed LED1: BLUE, led:LED3MM
- removed LED2, LED3: YELLOW, led:LED3MM
- removed R7L2, R8L3: 1k, rcl:0204/5
- removed X7, X9: NELTRON-7810-XPXC, con-rj45:NELTRON-7810-XPXC-FOOTPRINT
- added JP1, JP2: (no value), pinhead:1X06
- moved C5 63.0 mm to (14.0, 36.0)
- moved R9 44.1 mm to (20.0, 17.0)
- moved C4 40.3 mm to (24.0, 41.0)
- moved IC3 38.3 mm to (39.0, 33.5)
- moved LOGO1 37.3 mm to (8.50, 40.5)
- moved R2 35.0 mm to (11.2, 7.50)
- moved R1 34.4 mm to (8.61, 8.50)
- moved R3 33.6 mm to (14.7, 8.50)
- moved R4 32.0 mm to (19.2, 8.50)
- moved R5 31.6 mm to (20.8, 10.5)
- moved R6L1 30.2 mm to (24.3, 11.5)
- moved IC2 27.2 mm to (38.0, 20.5)
- moved RN2 11.4 mm to (36.5, 13.0)
Connections:
- removed net MTRTN: J8.5, R5.1
- removed net MTSND: J8.4, R4.1
- removed net N$1: IC1.6, LED2.K
- removed net N$2: LED3.A, R8L3.1
- removed net N$3: IC1.12, LED3.K
- removed net N$5: LED2.A, R7L2.1
- net GND: now also JP1.1, JP2.1; no longer J0.1, J0.2, J8.2, J9.2, LED1.K, X7.S1, X7.S2, X9.S1, X9.S2
- net MIRTN: now also JP1.4; no longer J7.5
- net MISND: now also JP1.3; no longer J7.4
- net MORTN: now also JP1.6; no longer J9.5
- net MOSND: now also JP1.5; no longer J9.4
- net N$4: now also JP2.2; no longer LED1.A
- net RX+: now also JP2.5; no longer X7.1
- net RX-: now also JP2.6; no longer X7.2
- net TX+: now also JP2.3; no longer X9.1
- net TX-: now also JP2.4; no longer X9.2
- net VCC: now also JP1.2; no longer J0.3, R7L2.2, R8L3.2
Routing:
- net GND: track 213.7 -> 0.00 mm, vias 1 -> 0
- net VCC: track 149.3 -> 0.00 mm
- net MIRTN: track 88.6 -> 0.00 mm
- net TX: track 88.0 -> 0.00 mm, vias 1 -> 0
- net N$3: track 66.9 -> 0.00 mm
- net N$1: track 66.0 -> 0.00 mm, vias 1 -> 0
- net RX: track 51.3 -> 0.00 mm
- net N$4: track 46.9 -> 0.00 mm
- net NMIDIOUT: track 40.6 -> 0.00 mm
- net MIDIIN: track 39.9 -> 0.00 mm
- net RX-: track 37.6 -> 0.00 mm
- net N$5: track 37.6 -> 0.00 mm
- net MISND: track 33.8 -> 0.00 mm
- net N$2: track 32.4 -> 0.00 mm
- net NMIDITHRU: track 30.1 -> 0.00 mm
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- removed copper zone on layer 1, net GND
- removed copper zone on layer 16, net GND
Other:
- board size 91 x 57 mm -> 47 x 47 mm

Commit message: First try.
Parts:
- removed R5: 220, rcl:0204/5
- R4: value 220 -> 100
- moved U$1 81.0 mm to (6.00, 31.0)
- moved R4 33.3 mm to (30.0, 40.0), turned to 0 degrees
- moved R2 32.9 mm to (38.0, 26.5)
- moved R3 32.7 mm to (42.0, 26.5)
- moved C5 28.1 mm to (16.0, 8.00)
- moved R6L1 27.6 mm to (38.0, 35.5)
- moved C4 25.0 mm to (23.5, 16.0), turned to 90 degrees
- moved C3 24.7 mm to (9.50, 16.0), turned to 90 degrees
- moved IC2 24.4 mm to (16.0, 31.0)
- moved R9 23.3 mm to (16.0, 40.0)
- moved LOGO1 22.7 mm to (23.5, 23.5)
- moved C1 19.8 mm to (9.50, 31.0), turned to 90 degrees
- moved C2 16.3 mm to (23.5, 31.0), turned to 90 degrees
- moved IC1 16.0 mm to (34.0, 16.0)
- moved OK1 14.8 mm to (16.0, 16.0)
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Connections:
- removed net MIDITHRU: IC1.4, R5.2
- removed net NMIDITHRU: IC1.2, IC1.3, RN2.3
- net GND: now also IC1.1, IC1.13, IC1.3, IC1.5
- net RX: no longer IC1.13
- net TX: no longer IC1.1, IC1.5
- net TX+: now also R4.1
- net TX-: now also R4.2
- net VCC: no longer R4.2
Routing:
- net GND: track 0.00 -> 121.9 mm
- net VCC: track 0.00 -> 106.2 mm
- net N$4: track 0.00 -> 38.6 mm
- net RX: track 0.00 -> 38.4 mm
- net TX: track 0.00 -> 37.8 mm
- net MORTN: track 0.00 -> 26.7 mm
- net MOSND: track 0.00 -> 26.4 mm
- net RX+: track 0.00 -> 23.8 mm
- net MISND: track 0.00 -> 23.4 mm
- net RX-: track 0.00 -> 22.7 mm
- net MIRTN: track 0.00 -> 22.4 mm
- net NMIDIOUT: track 0.00 -> 21.1 mm
- net TX-: track 0.00 -> 15.2 mm
- net TX+: track 0.00 -> 13.7 mm
- net MIDIIN: track 0.00 -> 13.6 mm
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Other:
- board text added: "4-M3"
- board text added: "Pineapple MiniMIDI 0.0.1-X"
- board text removed: "101"
- board text removed: "102"
- board text removed: "105"
- board text removed: "221"
- board text removed: "4-M2.3"
- board text removed: "472"
- board text removed: "7406"
- board text removed: "BLU"
- board text removed: "Designed for Takachi PF10-4-7"
- board text removed: "GRN"
- board text removed: "LTC485"
- board text removed: "MIDI IN"
- board text removed: "MIDI OUT"
- board text removed: "MIDI THRU"
- board text removed: "NC"
- board text removed: "NI"
- board text removed: "Neltron 7810-8P8C"
- board text removed: "OUT/THRU"
- board text removed: "Pineapple Zero 2.6.3-B"
- board text removed: "RX Terminator"
- board text removed: "TLP2630"
- board text removed: "YLW"

Commit message: Artwork.
Parts:
- JP2: device pinhead:1X06 -> pinhead:1X08
- moved RN2 16.0 mm to (34.0, 24.0)
- moved R6L1 6.73 mm to (43.0, 31.0)
- moved C5 5.83 mm to (13.0, 3.00)
- moved R3 4.92 mm to (40.0, 31.0)
- moved R2 4.61 mm to (37.0, 31.0)
- moved R4 2.00 mm to (30.0, 38.0)
- moved R9 2.00 mm to (16.0, 38.0)
Connections:
- new net V+: JP1.2, JP2.1
- net GND: now also JP2.3; no longer JP2.1
- net N$4: now also JP2.4; no longer JP2.2
- net RX+: now also JP2.7; no longer JP2.5
- net RX-: now also JP2.8; no longer JP2.6
- net TX+: now also JP2.5; no longer JP2.3
- net TX-: now also JP2.6; no longer JP2.4
- net VCC: now also JP2.2; no longer JP1.2
Routing:
- net V+: track 0.00 -> 49.9 mm
- net TX: track 37.8 -> 22.7 mm
- net NMIDIOUT: track 21.1 -> 11.8 mm
- net MOSND: track 26.4 -> 32.2 mm
- net RX: track 38.4 -> 33.7 mm
- net N$4: track 38.6 -> 42.4 mm
- net VCC: track 106.2 -> 109.9 mm
- net MIDIOUT: track 11.5 -> 15.2 mm
- net MORTN: track 26.7 -> 29.7 mm
- net MIRTN: track 22.4 -> 25.1 mm
- net TX-: track 15.2 -> 13.3 mm
- net RX+: track 23.8 -> 25.3 mm
- net RX-: track 22.7 -> 24.1 mm
- net TX+: track 13.7 -> 12.3 mm
- net GND: track 121.9 -> 121.0 mm, vias 0 -> 1
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
Commit message: Mostly done.
Parts:
- removed R6L1: 1k, rcl:0204/5
- removed RN2: 4.7k, resistor-net:RN-5
- added R6: 100, rcl:0204/5
- added RN1: 4.7k, resistor-net:RN-5
- C1: value 100n -> 10n
- C3: value 10n -> 100n
- JP1: value (none) -> Backside
- JP2: value (none) -> Frontside
- R4: value 100 -> 1k
- moved LOGO1 25.7 mm to (39.0, 3.00)
- moved U$1 19.5 mm to (23.5, 22.5), turned to 0 degrees
- moved C1 15.0 mm to (9.50, 16.0)
- moved C2 15.0 mm to (23.5, 16.0)
- moved C3 15.0 mm to (9.50, 31.0)
- moved C4 15.0 mm to (23.5, 31.0)
- moved R4 14.8 mm to (43.0, 31.0), turned to 90 degrees
- renumbered R9 to R5
Connections:
- removed net N$4: JP2.4, R6L1.1
- new net LED: JP2.4, R4.1
- net GND: now also JP2.1; no longer JP2.3
- net NMIDIOUT: now also RN1.5; no longer RN2.5
- net TX: now also RN1.2; no longer RN2.2
- net TX+: now also R6.1; no longer R4.1
- net TX-: now also R6.2; no longer R4.2
- net V+: now also JP2.2; no longer JP2.1
- net VCC: now also JP2.3, R4.2, RN1.1; no longer JP2.2, R6L1.2, RN2.1
Routing:
- net N$4: track 42.4 -> 0.00 mm
- net LED: track 0.00 -> 38.7 mm
- net NMIDIOUT: track 11.8 -> 45.7 mm, vias 0 -> 1
- net GND: track 121.0 -> 145.1 mm, vias 1 -> 0
- net VCC: track 109.9 -> 126.0 mm
- net TX: track 22.7 -> 36.6 mm
- net RX: track 33.7 -> 30.0 mm
- net MOSND: track 32.2 -> 29.5 mm
- net MIRTN: track 25.1 -> 22.4 mm
- net V+: track 49.9 -> 49.3 mm
- added copper zone on layer 1, net GND
- added copper zone on layer 16, net GND
Other:
- board text added: "Designed for Takachi MX2-6-10"
- board text added: "GND"
- board text added: "IN4"
- board text added: "IN5"
- board text added: "LED"
- board text added: "OUT4"
- board text added: "OUT5"
- board text added: "RX+"
- board text added: "RX-"
- board text added: "TX+"
- board text added: "TX-"
- board text added: "V+"
- board text added: "Vcc"
- board text removed: "IN"
- board text removed: "OUT"
- board text removed: "RX"
- board text removed: "THRU"
- board text removed: "TX"
